Commit message: add sound cam

File: URDF/box/box.urdf (robot description, URDF)
Before this commit: robot open_box, 6 links, 5 joints
Links:
- link back_plate: geometry collision box size=0.1 0.01 0.05; visual box size=0.1 0.01 0.05
- link bottom_plate: geometry collision box size=0.1 0.1 0.01; visual box size=0.1 0.1 0.01
- link front_plate: geometry collision box size=0.1 0.01 0.05; visual box size=0.1 0.01 0.05
- link left_plate: geometry collision box size=0.01 0.1 0.05; visual box size=0.01 0.1 0.05
- link right_plate: geometry collision box size=0.01 0.1 0.05; visual box size=0.01 0.1 0.05
Joints:
- joint bottom_to_back: origin xyz=0 -0.51 0 rpy=0 0 0 -> xyz=0 -0.051 0 rpy=0 0 0
- joint bottom_to_front: origin xyz=0 0.51 0 rpy=0 0 0 -> xyz=0 0.051 0 rpy=0 0 0
- joint bottom_to_left: origin xyz=-0.51 0 0 rpy=0 0 0 -> xyz=-0.051 0 0 rpy=0 0 0
- joint bottom_to_right: origin xyz=0.51 0 0 rpy=0 0 0 -> xyz=0.051 0 0 rpy=0 0 0
